File: pcb/kamstrup.sch (KiCad schematic (older format))
At the start: 11 parts, among them P1 CONN_4, Q1 BC557, Q2 BC547, Q3 BC547

Commit message: SMD version first commit
Parts:
- removed P1: CONN_4, symbol CONN_4
- removed Q1: BC557, TO92, symbol BC557
- removed Q2, Q3: BC547, TO92, symbol BC547
- added H1, H2: MountingHole, MountingHole:MountingHole_2.2mm_M2, symbol Mechanical:MountingHole
- added J1: GND, TestPoint:TestPoint_Pad_1.5x1.5mm, symbol Connector_Generic:Conn_01x01
- added J2: 5V, TestPoint:TestPoint_Pad_1.5x1.5mm, symbol Connector_Generic:Conn_01x01
- added J3: TX, TestPoint:TestPoint_Pad_1.5x1.5mm, symbol Connector_Generic:Conn_01x01
- added J4: RX, TestPoint:TestPoint_Pad_1.5x1.5mm, symbol Connector_Generic:Conn_01x01
- added Q1: PNP, Package_TO_SOT_SMD:SOT-23, symbol Device:Q_PNP_BEC
- added Q2, Q3: NPN, Package_TO_SOT_SMD:SOT-23, symbol Device:Q_NPN_BEC
- D1: renamed from TXLED1; value IR LED -> TX; footprint (none) -> LED_SMD:LED_0603_1608Metric; symbol LED_ALT -> Device:LED_ALT
- D2: renamed from RXLED1; value IR PHOTODIODE -> RX; footprint (none) -> LED_SMD:LED_0603_1608Metric; symbol D_Photo_ALT -> Device:D_Photo_ALT
- R1, R2, R3, R4, R5: footprint (none) -> Resistor_SMD:R_0603_1608Metric; symbol R-RESCUE-kamstrup -> kamstrup-rescue:R-RESCUE-kamstrup
Connections:
- net +5V: now also J2.1 (Pin_1), Q1.3 (C)
- net GND: now also J1.1 (Pin_1), Q3.2 (E)
- net RX: now also J4.1 (Pin_1), Q3.3 (C)
- net TX: now also J3.1 (Pin_1)
- net at R1.2: now also Q1.1 (B)
- net at R2.1: now also Q1.2 (E)
- net at R4.1: now also Q2.3 (C)
- net at D2.2 (A), R3.2: now also Q2.1 (B)
- new net: Q2.2 (E), Q3.1 (B)
Other:
- note added: "IR Phototransistor"
- note added: "IR led"
Changed lines of the file:
@@
-EESchema Schematic File Version 2
-LIBS:kamstrup-rescue
-LIBS:power
-LIBS:device
-LIBS:transistors
-LIBS:conn
-LIBS:linear
-LIBS:regul
-LIBS:74xx
-LIBS:cmos4000
-LIBS:adc-dac
-LIBS:memory
-LIBS:xilinx
-LIBS:microcontrollers
-LIBS:dsp
-LIBS:microchip
-LIBS:analog_switches
-LIBS:motorola
-LIBS:texas
-LIBS:intel
-LIBS:audio
-LIBS:interface
-LIBS:digital-audio
-LIBS:philips
-LIBS:display
-LIBS:cypress
-LIBS:siliconi
-LIBS:opto
-LIBS:atmel
-LIBS:contrib
-LIBS:valves
+EESchema Schematic File Version 4
 LIBS:kamstrup-cache
-EELAYER 25 0
+EELAYER 26 0
 EELAYER END
 $Descr User 8268 5827
@@
 	1450 3600 1900 3600
 Wire Wire Line
-	5100 2250 5100 2450
+	5100 2250 5100 2400
 Wire Wire Line
 	5100 2400 5350 2400
@@
 	6050 2900 6050 3100
 Wire Wire Line
-	6050 2150 6050 2500
+	6050 2150 6050 2350
 Wire Wire Line
 	5650 1550 5650 1650
@@
 TX
 $Comp
-L GND-RESCUE-kamstrup #PWR01
+L kamstrup-rescue:GND-RESCUE-kamstrup #PWR01
 U 1 1 51FBDA50
 P 5100 3100
@@
 $EndComp
 $Comp
-L R-RESCUE-kamstrup R4
+L kamstrup-rescue:R-RESCUE-kamstrup R4
 U 1 1 52CEFDF5
 P 5650 1900
 F 0 "R4" V 5730 1900 50  0000 C CNN
 F 1 "10k" V 5650 1900 50  0000 C CNN
-F 2 "" H 5650 1900 60  0001 C CNN
+F 2 "Resistor_SMD:R_0603_1608Metric" H 5650 1900 60  0001 C CNN
 F 3 "" H 5650 1900 60  0001 C CNN
 	1    5650 1900
@@
 $EndComp
 $Comp
-L R-RESCUE-kamstrup R5
+L kamstrup-rescue:R-RESCUE-kamstrup R5
 U 1 1 51FBDAB3
 P 6050 1900
 F 0 "R5" V 6130 1900 50  0000 C CNN
 F 1 "10k" V 6050 1900 50  0000 C CNN
-F 2 "" H 6050 1900 60  0001 C CNN
+F 2 "Resistor_SMD:R_0603_1608Metric" H 6050 1900 60  0001 C CNN
 F 3 "" H 6050 1900 60  0001 C CNN
 	1    6050 1900
@@
 $EndComp
 $Comp
-L BC547 Q3
-U 1 1 51FBDAA4
-P 5950 2700
-F 0 "Q3" H 5950 2551 40  0000 R CNN
-F 1 "BC547" H 5950 2850 40  0000 R CNN
-F 2 "TO92" H 5850 2802 29  0000 C CNN
-F 3 "" H 5950 2700 60  0001 C CNN
-	1    5950 2700
-	1    0    0    -1
-$EndComp
-$Comp
-L R-RESCUE-kamstrup R3
+L kamstrup-rescue:R-RESCUE-kamstrup R3
 U 1 1 51FBDA21
 P 5100 2700
 F 0 "R3" V 5180 2700 50  0000 C CNN
 F 1 "15k" V 5100 2700 50  0000 C CNN
-F 2 "" H 5100 2700 60  0001 C CNN
+F 2 "Resistor_SMD:R_0603_1608Metric" H 5100 2700 60  0001 C CNN
 F 3 "" H 5100 2700 60  0001 C CNN
 	1    5100 2700
@@
 TX
 $Comp
-L GND-RESCUE-kamstrup #PWR05
+L kamstrup-rescue:GND-RESCUE-kamstrup #PWR05
 U 1 1 51D5D924
 P 1800 3350
@@
 RX
 $Comp
-L BC547 Q2
-U 1 1 51D5D736
-P 5550 2400
-F 0 "Q2" H 5550 2251 40  0000 R CNN
-F 1 "BC547" H 5550 2550 40  0000 R CNN
-F 2 "TO92" H 5450 2502 29  0000 C CNN
-F 3 "" H 5550 2400 60  0001 C CNN
-	1    5550 2400
-	1    0    0    -1
-$EndComp
-$Comp
-L GND-RESCUE-kamstrup #PWR06
+L kamstrup-rescue:GND-RESCUE-kamstrup #PWR06
 U 1 1 51D5D72C
 P 6050 3100
@@
 $EndComp
 $Comp
-L R-RESCUE-kamstrup R2
+L kamstrup-rescue:R-RESCUE-kamstrup R2
 U 1 1 51D5D6E0
 P 2650 2400
 F 0 "R2" V 2730 2400 50  0000 C CNN
 F 1 "220" V 2650 2400 50  0000 C CNN
-F 2 "" H 2650 2400 60  0001 C CNN
+F 2 "Resistor_SMD:R_0603_1608Metric" H 2650 2400 60  0001 C CNN
 F 3 "" H 2650 2400 60  0001 C CNN
 	1    2650 2400
@@
 $EndComp
 $Comp
-L CONN_4 P1
-U 1 1 51D5D6C3
-P 1100 3450
-F 0 "P1" V 1050 3450 50  0000 C CNN
-F 1 "CONN_4" V 1150 3450 50  0000 C CNN
-F 2 "" H 1100 3450 60  0001 C CNN
-F 3 "" H 1100 3450 60  0001 C CNN
-	1    1100 3450
-	-1   0    0    1
-$EndComp
-$Comp
-L BC557 Q1
-U 1 1 51D5D65F
-P 2550 1900
-F 0 "Q1" H 2550 1751 40  0000 R CNN
-F 1 "BC557" H 2550 2050 40  0000 R CNN
-F 2 "TO92" H 2450 2002 29  0000 C CNN
-F 3 "" H 2550 1900 60  0001 C CNN
-	1    2550 1900
-	1    0    0    1
-$EndComp
-$Comp
-L R-RESCUE-kamstrup R1
+L kamstrup-rescue:R-RESCUE-kamstrup R1
 U 1 1 51D5D637
 P 1950 1900
 F 0 "R1" V 2030 1900 50  0000 C CNN
 F 1 "39k" V 1950 1900 50  0000 C CNN
-F 2 "" H 1950 1900 60  0001 C CNN
+F 2 "Resistor_SMD:R_0603_1608Metric" H 1950 1900 60  0001 C CNN
 F 3 "" H 1950 1900 60  0001 C CNN
 	1    1950 1900
@@
 $EndComp
 $Comp
-L GND-RESCUE-kamstrup #PWR08
+L kamstrup-rescue:GND-RESCUE-kamstrup #PWR08
 U 1 1 51D5D613
 P 2650 3350
@@
 $EndComp
 $Comp
-L LED_ALT TXLED1
+L Device:LED_ALT D1
 U 1 1 59706A67
 P 2650 2850
-F 0 "TXLED1" H 2650 2950 50  0000 C CNN
-F 1 "IR LED" H 2650 2750 50  0000 C CNN
-F 2 "" H 2650 2850 50  0001 C CNN
+F 0 "D1" H 2650 2950 50  0000 C CNN
+F 1 "TX" H 2650 2750 50  0000 C CNN
+F 2 "LED_SMD:LED_0603_1608Metric" H 2650 2850 50  0001 C CNN
 F 3 "" H 2650 2850 50  0001 C CNN
 	1    2650 2850
@@
 $EndComp
 $Comp
-L D_Photo_ALT RXLED1
+L Device:D_Photo_ALT D2
 U 1 1 59706C4F
 P 5100 2150
-F 0 "RXLED1" H 5120 2220 50  0000 L CNN
-F 1 "IR PHOTODIODE" H 5060 2040 50  0000 C CNN
-F 2 "" H 5050 2150 50  0001 C CNN
+F 0 "D2" H 5120 2220 50  0000 L CNN
+F 1 "RX" H 5060 2040 50  0000 C CNN
+F 2 "LED_SMD:LED_0603_1608Metric" H 5050 2150 50  0001 C CNN
 F 3 "" H 5050 2150 50  0001 C CNN
 	1    5100 2150
@@
 $EndComp
 $Comp
-L +5V #PWR?
+L power:+5V #PWR0101
 U 1 1 59706D36
 P 2650 1500
-F 0 "#PWR?" H 2650 1350 50  0001 C CNN
+F 0 "#PWR0101" H 2650 1350 50  0001 C CNN
 F 1 "+5V" H 2650 1640 50  0000 C CNN
 F 2 "" H 2650 1500 50  0001 C CNN
@@
 $EndComp
 $Comp
-L +5V #PWR?
+L power:+5V #PWR0102
 U 1 1 59706D6F
 P 1600 3200
-F 0 "#PWR?" H 1600 3050 50  0001 C CNN
+F 0 "#PWR0102" H 1600 3050 50  0001 C CNN
 F 1 "+5V" H 1600 3340 50  0000 C CNN
 F 2 "" H 1600 3200 50  0001 C CNN
@@
 	1600 3400 1600 3200
 $Comp
-L +5V #PWR?
+L power:+5V #PWR0103
 U 1 1 59706DE7
 P 5650 1550
-F 0 "#PWR?" H 5650 1400 50  0001 C CNN
+F 0 "#PWR0103" H 5650 1400 50  0001 C CNN
 F 1 "+5V" H 5650 1690 50  0000 C CNN
 F 2 "" H 5650 1550 50  0001 C CNN
@@
 $EndComp
 $Comp
-L +5V #PWR?
+L power:+5V #PWR0104
 U 1 1 59706E11
 P 6050 1550
-F 0 "#PWR?" H 6050 1400 50  0001 C CNN
+F 0 "#PWR0104" H 6050 1400 50  0001 C CNN
 F 1 "+5V" H 6050 1690 50  0000 C CNN
 F 2 "" H 6050 1550 50  0001 C CNN
@@
 Wire Wire Line
 	5100 1650 5100 1950
+Wire Wire Line
+	6050 2350 6050 2500
+Wire Wire Line
+	5100 2400 5100 2450
+$Comp
+L Device:Q_PNP_BEC Q1
+U 1 1 5C8CDC16
+P 2550 1900
+F 0 "Q1" H 2741 1946 50  0000 L CNN
+F 1 "PNP" H 2741 1855 50  0000 L CNN
+F 2 "Package_TO_SOT_SMD:SOT-23" H 2750 2000 50  0001 C CNN
+F 3 "~" H 2550 1900 50  0001 C CNN
+	1    2550 1900
+	1    0    0    -1
+$EndComp
+$Comp
+L Device:Q_NPN_BEC Q2
+U 1 1 5C8CDE9E
+P 5550 2400
+F 0 "Q2" H 5741 2446 50  0000 L CNN
+F 1 "NPN" H 5741 2355 50  0000 L CNN
+F 2 "Package_TO_SOT_SMD:SOT-23" H 5750 2500 50  0001 C CNN
+F 3 "~" H 5550 2400 50  0001 C CNN
+	1    5550 2400
+	1    0    0    -1
+$EndComp
+$Comp
+L Device:Q_NPN_BEC Q3
+U 1 1 5C8CDF18
+P 5950 2700
+F 0 "Q3" H 6141 2746 50  0000 L CNN
+F 1 "NPN" H 6141 2655 50  0000 L CNN
+F 2 "Package_TO_SOT_SMD:SOT-23" H 6150 2800 50  0001 C CNN
+F 3 "~" H 5950 2700 50  0001 C CNN
+	1    5950 2700
+	1    0    0    -1
+$EndComp
+$Comp
+L Mechanical:MountingHole H1
+U 1 1 5C93F3AA
+P 1100 4200
+F 0 "H1" H 1200 4246 50  0000 L CNN
+F 1 "MountingHole" H 1200 4155 50  0000 L CNN
+F 2 "MountingHole:MountingHole_2.2mm_M2" H 1100 4200 50  0001 C CNN
+F 3 "~" H 1100 4200 50  0001 C CNN
+	1    1100 4200
+	1    0    0    -1
+$EndComp
+$Comp
+L Mechanical:MountingHole H2
+U 1 1 5C93F4E8
+P 1100 4450
+F 0 "H2" H 1200 4496 50  0000 L CNN
+F 1 "MountingHole" H 1200 4405 50  0000 L CNN
+F 2 "MountingHole:MountingHole_2.2mm_M2" H 1100 4450 50  0001 C CNN
+F 3 "~" H 1100 4450 50  0001 C CNN
+	1    1100 4450
+	1    0    0    -1
+$EndComp
+$Comp
+L Connector_Generic:Conn_01x01 J1
+U 1 1 5C93FBE8
+P 1250 3300
+F 0 "J1" H 1170 3075 50  0000 C CNN
+F 1 "GND" H 1170 3166 50  0000 C CNN
+F 2 "TestPoint:TestPoint_Pad_1.5x1.5mm" H 1250 3300 50  0001 C CNN
+F 3 "~" H 1250 3300 50  0001 C CNN
+	1    1250 3300
+	-1   0    0    1
+$EndComp
+$Comp
+L Connector_Generic:Conn_01x01 J2
+U 1 1 5C93FC78
+P 1250 3400
+F 0 "J2" H 1170 3175 50  0000 C CNN
+F 1 "5V" H 1170 3266 50  0000 C CNN
+F 2 "TestPoint:TestPoint_Pad_1.5x1.5mm" H 1250 3400 50  0001 C CNN
+F 3 "~" H 1250 3400 50  0001 C CNN
+	1    1250 3400
+	-1   0    0    1
+$EndComp
+$Comp
+L Connector_Generic:Conn_01x01 J3
+U 1 1 5C93FCA4
+P 1250 3500
+F 0 "J3" H 1170 3275 50  0000 C CNN
+F 1 "TX" H 1170 3366 50  0000 C CNN
+F 2 "TestPoint:TestPoint_Pad_1.5x1.5mm" H 1250 3500 50  0001 C CNN
+F 3 "~" H 1250 3500 50  0001 C CNN
+	1    1250 3500
+	-1   0    0    1
+$EndComp
+$Comp
+L Connector_Generic:Conn_01x01 J4
+U 1 1 5C93FCD2
+P 1250 3600
+F 0 "J4" H 1170 3375 50  0000 C CNN
+F 1 "RX" H 1170 3466 50  0000 C CNN
+F 2 "TestPoint:TestPoint_Pad_1.5x1.5mm" H 1250 3600 50  0001 C CNN
+F 3 "~" H 1250 3600 50  0001 C CNN
+	1    1250 3600
+	-1   0    0    1
+$EndComp
+Text Notes 4950 2600 1    60   ~ 0
+IR Phototransistor
+Text Notes 2500 3000 1    60   ~ 0
+IR led
 $EndSCHEMATC

Commit message: Clean up and gerber files for pcb
Parts:
- R1, R2, R3, R4, R5: symbol kamstrup-rescue:R-RESCUE-kamstrup -> Device:R
Changed lines of the file:
@@
 Text Notes 3900 1500 0    60   ~ 0
 Echo cancellation:\nTX is high when inactive,\nso only let the LED \nreceive when TX is high.
-Wire Wire Line
-	5650 2150 5650 2200
 Connection ~ 6050 2350
 Wire Wire Line
 	6050 2350 6350 2350
 Wire Wire Line
-	6050 1550 6050 1650
-Wire Wire Line
 	5750 2700 5650 2700
 Wire Wire Line
 	5650 2700 5650 2600
 Wire Wire Line
-	5100 2950 5100 3100
-Wire Wire Line
 	1650 3500 1450 3500
 Wire Wire Line
-	1800 3350 1800 3300
-Wire Wire Line
-	1800 3300 1450 3300
-Wire Wire Line
-	2650 2650 2650 2700
-Wire Wire Line
-	2350 1900 2200 1900
-Wire Wire Line
 	2650 1700 2650 1500
 Wire Wire Line
-	2650 2150 2650 2100
-Wire Wire Line
 	2650 3000 2650 3350
-Wire Wire Line
-	1450 1900 1700 1900
 Wire Wire Line
 	1450 3400 1600 3400
@@
 Wire Wire Line
 	6050 2900 6050 3100
-Wire Wire Line
-	6050 2150 6050 2350
-Wire Wire Line
-	5650 1550 5650 1650
 Text GLabel 4650 1650 0    60   Input ~ 0
 TX
 $Comp
-L kamstrup-rescue:GND-RESCUE-kamstrup #PWR01
-U 1 1 51FBDA50
-P 5100 3100
-F 0 "#PWR01" H 5100 3100 30  0001 C CNN
-F 1 "GND" H 5100 3030 30  0001 C CNN
-F 2 "" H 5100 3100 60  0001 C CNN
-F 3 "" H 5100 3100 60  0001 C CNN
-	1    5100 3100
-	1    0    0    -1
-$EndComp
-$Comp
-L kamstrup-rescue:R-RESCUE-kamstrup R4
+L Device:R R4
 U 1 1 52CEFDF5
 P 5650 1900
@@
 $EndComp
 $Comp
-L kamstrup-rescue:R-RESCUE-kamstrup R5
+L Device:R R5
 U 1 1 51FBDAB3
 P 6050 1900
@@
 $EndComp
 $Comp
-L kamstrup-rescue:R-RESCUE-kamstrup R3
+L Device:R R3
 U 1 1 51FBDA21
 P 5100 2700
@@
 Text GLabel 1650 3500 2    60   Input ~ 0
 TX
-$Comp
-L kamstrup-rescue:GND-RESCUE-kamstrup #PWR05
-U 1 1 51D5D924
-P 1800 3350
-F 0 "#PWR05" H 1800 3350 30  0001 C CNN
-F 1 "GND" H 1800 3280 30  0001 C CNN
-F 2 "" H 1800 3350 60  0001 C CNN
-F 3 "" H 1800 3350 60  0001 C CNN
-	1    1800 3350
-	1    0    0    -1
-$EndComp
 Text GLabel 1450 1900 0    60   Input ~ 0
 TX
@@
 RX
 $Comp
-L kamstrup-rescue:GND-RESCUE-kamstrup #PWR06
-U 1 1 51D5D72C
-P 6050 3100
-F 0 "#PWR06" H 6050 3100 30  0001 C CNN
-F 1 "GND" H 6050 3030 30  0001 C CNN
-F 2 "" H 6050 3100 60  0001 C CNN
-F 3 "" H 6050 3100 60  0001 C CNN
-	1    6050 3100
-	1    0    0    -1
-$EndComp
-$Comp
-L kamstrup-rescue:R-RESCUE-kamstrup R2
+L Device:R R2
 U 1 1 51D5D6E0
 P 2650 2400
@@
 $EndComp
 $Comp
-L kamstrup-rescue:R-RESCUE-kamstrup R1
+L Device:R R1
 U 1 1 51D5D637
 P 1950 1900
@@
 	1    1950 1900
 	0    -1   -1   0
-$EndComp
-$Comp
-L kamstrup-rescue:GND-RESCUE-kamstrup #PWR08
-U 1 1 51D5D613
-P 2650 3350
-F 0 "#PWR08" H 2650 3350 30  0001 C CNN
-F 1 "GND" H 2650 3280 30  0001 C CNN
-F 2 "" H 2650 3350 60  0001 C CNN
-F 3 "" H 2650 3350 60  0001 C CNN
-	1    2650 3350
-	1    0    0    -1
 $EndComp
 $Comp
@@
 Wire Wire Line
 	6050 2350 6050 2500
-Wire Wire Line
-	5100 2400 5100 2450
 $Comp
 L Device:Q_PNP_BEC Q1
@@
 Text Notes 2500 3000 1    60   ~ 0
 IR led
+Wire Wire Line
+	2100 1900 2350 1900
+Wire Wire Line
+	1450 1900 1800 1900
+Wire Wire Line
+	2650 2550 2650 2700
+Wire Wire Line
+	2650 2100 2650 2250
+Wire Wire Line
+	6050 2050 6050 2350
+Wire Wire Line
+	5650 2050 5650 2200
+Wire Wire Line
+	5650 1550 5650 1750
+Wire Wire Line
+	6050 1550 6050 1750
+Wire Wire Line
+	5100 2400 5100 2550
+Wire Wire Line
+	5100 2850 5100 3100
+$Comp
+L power:GND #PWR?
+U 1 1 5C968C45
+P 2050 3300
+F 0 "#PWR?" H 2050 3050 50  0001 C CNN
+F 1 "GND" H 2055 3127 50  0000 C CNN
+F 2 "" H 2050 3300 50  0001 C CNN
+F 3 "" H 2050 3300 50  0001 C CNN
+	1    2050 3300
+	1    0    0    -1
+$EndComp
+$Comp
+L power:GND #PWR?
+U 1 1 5C968C97
+P 2650 3350
+F 0 "#PWR?" H 2650 3100 50  0001 C CNN
+F 1 "GND" H 2655 3177 50  0000 C CNN
+F 2 "" H 2650 3350 50  0001 C CNN
+F 3 "" H 2650 3350 50  0001 C CNN
+	1    2650 3350
+	1    0    0    -1
+$EndComp
+$Comp
+L power:GND #PWR?
+U 1 1 5C968CC2
+P 5100 3100
+F 0 "#PWR?" H 5100 2850 50  0001 C CNN
+F 1 "GND" H 5105 2927 50  0000 C CNN
+F 2 "" H 5100 3100 50  0001 C CNN
+F 3 "" H 5100 3100 50  0001 C CNN
+	1    5100 3100
+	1    0    0    -1
+$EndComp
+$Comp
+L power:GND #PWR?
+U 1 1 5C968D2D
+P 6050 3100
+F 0 "#PWR?" H 6050 2850 50  0001 C CNN
+F 1 "GND" H 6055 2927 50  0000 C CNN
+F 2 "" H 6050 3100 50  0001 C CNN
+F 3 "" H 6050 3100 50  0001 C CNN
+	1    6050 3100
+	1    0    0    -1
+$EndComp
+Wire Wire Line
+	1450 3300 2050 3300
 $EndSCHEMATC

Commit message: Added link to datasheet for components.
Parts:
- D1: Type (none) -> APT1608F3C
- D2: Type (none) -> EAPST1608A0
- Q1: Type (none) -> MMBT3906
- Q2, Q3: Type (none) -> MMBT3904
Changed lines of the file:
@@
 Sheet 1 1
 Title "Kamstrup IR-head"
-Date "20 Jul 2017"
-Rev "2"
+Date "2019-03-23"
+Rev "3"
 Comp ""
 Comment1 ""
@@
 F 1 "TX" H 2650 2750 50  0000 C CNN
 F 2 "LED_SMD:LED_0603_1608Metric" H 2650 2850 50  0001 C CNN
-F 3 "" H 2650 2850 50  0001 C CNN
+F 3 "http://static6.arrow.com/aropdfconversion/e52aea5d9055317c3ce7432ccd22a4384016af9/3421969660189984apt1608f3c.pdf" H 2650 2850 50  0001 C CNN
+F 4 "APT1608F3C" H 2650 2850 50  0001 C CNN "Type"
 	1    2650 2850
 	0    -1   -1   0
@@
 F 1 "RX" H 5060 2040 50  0000 C CNN
 F 2 "LED_SMD:LED_0603_1608Metric" H 5050 2150 50  0001 C CNN
-F 3 "" H 5050 2150 50  0001 C CNN
+F 3 "http://static6.arrow.com/aropdfconversion/2325fc502e23b537918014f6f2d82469c984eab0/401index.phptrollerattachmentid_attachment820.phptrollerattach.pdf" H 5050 2150 50  0001 C CNN
+F 4 "EAPST1608A0" H 5100 2150 50  0001 C CNN "Type"
 	1    5100 2150
 	0    -1   1    0
@@
 F 1 "PNP" H 2741 1855 50  0000 L CNN
 F 2 "Package_TO_SOT_SMD:SOT-23" H 2750 2000 50  0001 C CNN
-F 3 "~" H 2550 1900 50  0001 C CNN
+F 3 "https://assets.nexperia.com/documents/data-sheet/MMBT3906.pdf" H 2550 1900 50  0001 C CNN
+F 4 "MMBT3906" H 2550 1900 50  0001 C CNN "Type"
 	1    2550 1900
 	1    0    0    -1
@@
 F 1 "NPN" H 5741 2355 50  0000 L CNN
 F 2 "Package_TO_SOT_SMD:SOT-23" H 5750 2500 50  0001 C CNN
-F 3 "~" H 5550 2400 50  0001 C CNN
+F 3 "https://www.diodes.com/assets/Datasheets/ds30036.pdf" H 5550 2400 50  0001 C CNN
+F 4 "MMBT3904" H 5550 2400 50  0001 C CNN "Type"
 	1    5550 2400
 	1    0    0    -1
@@
 F 1 "NPN" H 6141 2655 50  0000 L CNN
 F 2 "Package_TO_SOT_SMD:SOT-23" H 6150 2800 50  0001 C CNN
-F 3 "~" H 5950 2700 50  0001 C CNN
+F 3 "https://www.diodes.com/assets/Datasheets/ds30036.pdf" H 5950 2700 50  0001 C CNN
+F 4 "MMBT3904" H 5950 2700 50  0001 C CNN "Type"
 	1    5950 2700
 	1    0    0    -1
